File: PCB/ToolChanger/ToolChanger.kicad_pcb (KiCad board)
At the start: 2 copper layers, 139.7 x 80 mm, 23 parts, among them J1 Conn_01x26_Male, J2 Con_Motor, J3 Conn_01x06, J4 Conn_01x02, U1 STM32L-Discovery, U2 PC817, U3 PC817, U4 PC817, U5 PC817

Commit message: Initial commit. Toolchange working
Other:
- board text added: "10"
- board text added: "9"
Changed lines of the file:
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@@
   (general
     (thickness 1.6)
-    (drawings 12)
+    (drawings 16)
     (tracks 158)
     (zones 0)
@@
   )
   (setup
-    (last_trace_width 0.5)
+    (last_trace_width 0.25)
     (user_trace_width 0.25)
     (user_trace_width 0.5)
@@
       (net 31 +5V))
   )
+  (gr_text 2 (at 163.83762 91.88958) (layer F.SilkS)
+    (effects (font (size 1.5 1.5) (thickness 0.3)))
+  )
+  (gr_text 9 (at 174.0916 103.79964) (layer F.SilkS)
+    (effects (font (size 1.5 1.5) (thickness 0.3)))
+  )
+  (gr_text 10 (at 174.79264 91.98356) (layer F.SilkS)
+    (effects (font (size 1.5 1.5) (thickness 0.3)))
+  )
+  (gr_text 1 (at 163.5506 103.89362) (layer F.SilkS)
+    (effects (font (size 1.5 1.5) (thickness 0.3)))
+  )
   (gr_text +24 (at 208.5086 81.0768 90) (layer F.SilkS)
